Commit message: Section 9 - Odometry - complete

File: src/bumperbot_description/urdf/bumperbot_ros2_control.xacro (robot description, xacro)
@@ -6,5 +6,5 @@
             </hardware>
         </xacro:if>
-        <joint name="wheel_left_joint" type="revolute">
+        <joint name="wheel_right_joint" type="revolute">
             <command_interface name="velocity">
                 <param name="min">-1</param>
@@ -14,5 +14,5 @@
             <state_interface name="velocity"/>
         </joint>
-        <joint name="wheel_right_joint" type="revolute">
+        <joint name="wheel_left_joint" type="revolute">
             <command_interface name="velocity">
                 <param name="min">-1</param>

Commit message: using the ros2 ekf library

File: src/bumperbot_description/urdf/bumperbot_ros2_control.xacro (robot description, xacro)
@@ -6,5 +6,5 @@
             </xacro:if>
         </hardware>
-        <joint name="wheel_right_joint" type="revolute">
+        <joint name="wheel_right_joint">
             <command_interface name="velocity">
                 <param name="min">-1</param>
@@ -14,5 +14,5 @@
             <state_interface name="velocity" />
         </joint>
-        <joint name="wheel_left_joint" type="revolute">
+        <joint name="wheel_left_joint">
             <command_interface name="velocity">
                 <param name="min">-1</param>
