Commit message: End Section 4

File: src/bumperbot_description/urdf/bumperbot.urdf.xacro (robot description, xacro)
@@ -1,2 +1,159 @@
-<robot name="bumperbot">
+<robot name="bumperbot" xmlns:xacro="http://www.ros.org/wiki/xacro">
+    <xacro:property name="PI" value="3.14159" />
+    <xacro:property name="effort" value="30.0" />
+    <xacro:property name="velocity" value="10.0" />
+    <xacro:macro name="default_inertial" params="mass">
+        <inertial>
+            <mass value="${mass}" />
+            <inertia ixx="1.0" ixy="0.0" ixz="0.0"
+                iyy="1.0" iyz="0.0"
+                izz="1.0" />
+        </inertial>
+    </xacro:macro>
+    <xacro:include filename="$(find bumperbot_description)/urdf/colors.xacro" />
+    <xacro:include filename="$(find bumperbot_description)/urdf/bumperbot_gazebo.xacro" />
+    <!-- <xacro:include filename="$(find bumperbot_description)/urdf/can.xacro" /> -->
+    <link name="base_footprint" />
+    <link name="base_link">
+        <inertial>
+            <origin xyz="0 0 0.04" rpy="0.0 0.25 0.3" />
+            <mass value="8.2573504e-01" />
+            <inertia ixx="2.2124416e-02" ixy="-1.2294101e-04" ixz="3.4938785e-04"
+                iyy="2.1193702e-02" iyz="-5.0120904e-05"
+                izz="2.0064271e-02" />
+        </inertial>
+        <visual>
+            <origin rpy="0 0 0" xyz="0 0 0" />
+            <geometry>
+                <mesh filename="package://bumperbot_description/meshes/base_link.STL" />
+            </geometry>
+            <material name="purple" />
+        </visual>
+        <collision>
+            <origin rpy="0 0 0" xyz="0 0 0" />
+            <geometry>
+                <mesh filename="package://bumperbot_description/meshes/base_link.STL" />
+            </geometry>
+        </collision>
+    </link>
+    <link name="wheel_right_link">
+        <inertial>
+            <origin xyz="0 -0.014 0" rpy="0 0 0" />
+            <mass value="0.0530086090966721" />
+            <inertia ixx="1.88176298336665E-05" ixy="-4.8444933029987E-10"
+                ixz="1.88163708851143E-08"
+                iyy="3.11510738647764E-05" iyz="-6.93560663069607E-11"
+                izz="1.8801969558182E-05" />
+        </inertial>
+        <visual>
+            <origin rpy="-${PI/2} 0 0" xyz="0 0 0" />
+            <geometry>
+                <mesh filename="package://bumperbot_description/meshes/wheel_right_link.STL" />
+            </geometry>
+            <material name="black" />
+        </visual>
+        <collision>
+            <origin rpy="-${PI/2} 0 0" xyz="0 0 0" />
+            <geometry>
+                <mesh filename="package://bumperbot_description/meshes/wheel_right_link.STL" />
+            </geometry>
+        </collision>
+    </link>
+    <link name="wheel_left_link">
+        <inertial>
+            <origin xyz="0 0.014 0" rpy="0 0 0" />
+            <mass value="0.0530086043217644" />
+            <inertia ixx="1.8792911368909E-05" ixy="3.31256392204584E-10"
+                ixz="-1.14082001662767E-08"
+                iyy="3.11510738759073E-05" iyz="-3.60499245082192E-10"
+                izz="1.88266886146847E-05" />
+        </inertial>
+        <visual>
+            <origin rpy="${PI/2} 0 0" xyz="0 0 0" />
+            <geometry>
+                <mesh filename="package://bumperbot_description/meshes/wheel_left_link.STL" />
+            </geometry>
+            <material name="black" />
+        </visual>
+        <collision>
+            <origin rpy="${PI/2} 0 0" xyz="0 0 0" />
+            <geometry>
+                <mesh filename="package://bumperbot_description/meshes/wheel_left_link.STL" />
+            </geometry>
+        </collision>
+    </link>
+    <link name="caster_front_link">
+        <inertial>
+            <origin xyz="3.89968128948481E-07 2.40073004698083E-07 0.00219173397061506" rpy="0 0 0" />
+            <mass value="1.44379265037903E-06" />
+            <inertia ixx="7.23075276010246E-11" ixy="-6.10956883467859E-16"
+                ixz="2.22849693525031E-15"
+                iyy="3.8713793085917E-11" iyz="2.93909858781952E-15"
+                izz="1.00967486676306E-10" />
+        </inertial>
+        <visual>
+            <origin rpy="0 0 0" xyz="0 0 0" />
+            <geometry>
+                <mesh filename="package://bumperbot_description/meshes/caster_front_link.STL" />
+            </geometry>
+            <material name="black" />
+        </visual>
+        <collision>
+            <origin rpy="-0 0 0" xyz="0 0 0" />
+            <geometry>
+                <mesh filename="package://bumperbot_description/meshes/caster_front_link.STL" />
+            </geometry>
+        </collision>
+    </link>
+    <link name="caster_rear_link">
+        <inertial>
+            <origin xyz="3.8996812895542E-07 2.40073004698083E-07 0.00219173397061509" rpy="0 0 0" />
+            <mass value="1.44379265037902E-06" />
+            <inertia ixx="7.23075276010246E-11" ixy="-6.10956872363424E-16"
+                ixz="2.22849693527207E-15"
+                iyy="3.87137930859167E-11" iyz="2.939098587861E-15"
+                izz="1.00967486676306E-10" />
+        </inertial>
+        <visual>
+            <origin rpy="0 0 0" xyz="0 0 0" />
+            <geometry>
+                <mesh filename="package://bumperbot_description/meshes/caster_rear_link.STL" />
+            </geometry>
+            <material name="black" />
+        </visual>
+        <collision>
+            <origin rpy="-0 0 0" xyz="0 0 0" />
+            <geometry>
+                <mesh filename="package://bumperbot_description/meshes/caster_rear_link.STL" />
+            </geometry>
+        </collision>
+    </link>
+    <!-- JOINTS -->
+    <joint name="base_joint" type="fixed">
+        <parent link="base_footprint" />
+        <child link="base_link" />
+        <origin rpy="0 0 0" xyz="0 0 0.033" />
+    </joint>
+    <joint name="wheel_right_joint" type="continuous">
+        <parent link="base_link" />
+        <child link="wheel_right_link" />
+        <origin rpy="0 0 0" xyz="0 0.07 0.0" />
+        <axis xyz="0 1 0" />
+    </joint>
+    <joint name="wheel_left_joint" type="continuous">
+        <parent link="base_link" />
+        <child link="wheel_left_link" />
+        <origin rpy="0 0 0" xyz="0 -0.07 0.0" />
+        <axis xyz="0 1 0" />
+    </joint>
+    <joint name="caster_front_joint" type="fixed">
+        <parent link="base_link" />
+        <child link="caster_front_link" />
+        <origin rpy="0 0 0" xyz="0.04755 0 -0.0275" />
+    </joint>
+    <joint name="caster_rear_joint" type="fixed">
+        <parent link="base_link" />
+        <child link="caster_rear_link" />
+        <origin rpy="0 0 0" xyz="-0.04755 0  -0.0275" />
+    </joint>
 </robot>

Commit message: end section 5

File: src/bumperbot_description/urdf/bumperbot.urdf.xacro (robot description, xacro)
@@ -1,14 +1,7 @@
 <robot name="bumperbot" xmlns:xacro="http://www.ros.org/wiki/xacro">
+    <xacro:arg name="is_sim" default="true" />
     <xacro:property name="PI" value="3.14159" />
     <xacro:property name="effort" value="30.0" />
     <xacro:property name="velocity" value="10.0" />
-    <xacro:macro name="default_inertial" params="mass">
-        <inertial>
-            <mass value="${mass}" />
-            <inertia ixx="1.0" ixy="0.0" ixz="0.0"
-                iyy="1.0" iyz="0.0"
-                izz="1.0" />
-        </inertial>
-    </xacro:macro>
     <xacro:include filename="$(find bumperbot_description)/urdf/colors.xacro" />
     <xacro:include filename="$(find bumperbot_description)/urdf/bumperbot_gazebo.xacro" />
@@ -52,10 +45,10 @@
                 <mesh filename="package://bumperbot_description/meshes/wheel_right_link.STL" />
             </geometry>
-            <material name="black" />
+            <material name="green" />
         </visual>
         <collision>
-            <origin rpy="-${PI/2} 0 0" xyz="0 0 0" />
+            <origin xyz="0 -0.015 0" rpy="1.57 0 0" />
             <geometry>
-                <mesh filename="package://bumperbot_description/meshes/wheel_right_link.STL" />
+                <sphere radius="0.033" />
             </geometry>
         </collision>
@@ -75,10 +68,10 @@
                 <mesh filename="package://bumperbot_description/meshes/wheel_left_link.STL" />
             </geometry>
-            <material name="black" />
+            <material name="red" />
         </visual>
         <collision>
-            <origin rpy="${PI/2} 0 0" xyz="0 0 0" />
+            <origin xyz="0 0.015 0" rpy="-1.57 0 0" />
             <geometry>
-                <mesh filename="package://bumperbot_description/meshes/wheel_left_link.STL" />
+                <sphere radius="0.033" />
             </geometry>
         </collision>
@@ -101,7 +94,7 @@
         </visual>
         <collision>
-            <origin rpy="-0 0 0" xyz="0 0 0" />
+            <origin xyz="0 0 0" rpy="0 0 0" />
             <geometry>
-                <mesh filename="package://bumperbot_description/meshes/caster_front_link.STL" />
+                <sphere radius="0.005" />
             </geometry>
         </collision>
@@ -124,7 +117,7 @@
         </visual>
         <collision>
-            <origin rpy="-0 0 0" xyz="0 0 0" />
+            <origin xyz="0 0 0" rpy="0 0 0" />
             <geometry>
-                <mesh filename="package://bumperbot_description/meshes/caster_rear_link.STL" />
+                <sphere radius="0.005" />
             </geometry>
         </collision>

File: src/bumperbot_description/urdf/bumperbot_gazebo.xacro (robot description, xacro)
@@ -1,8 +1,8 @@
 <robot xmlns:xacro="http://www.ros.org/wiki/xacro">
     <gazebo reference="wheel_right_link">
-        <mu1>1e+14</mu1>
-        <mu2>1e+14</mu2>
-        <kp>1e+12</kp>
-        <kd>10</kd>
+        <mu1>1000000000000000.0</mu1>
+        <mu2>1000000000000000.0</mu2>
+        <kp>1000000000000.0</kp>
+        <kd>10.0</kd>
         <minDepth>0.001</minDepth>
         <maxVel>0.1</maxVel>
@@ -10,8 +10,8 @@
     </gazebo>
     <gazebo reference="wheel_left_link">
-        <mu1>1e+14</mu1>
-        <mu2>1e+14</mu2>
-        <kp>1e+12</kp>
-        <kd>10</kd>
+        <mu1>1000000000000000.0</mu1>
+        <mu2>1000000000000000.0</mu2>
+        <kp>1000000000000.0</kp>
+        <kd>10.0</kd>
         <minDepth>0.001</minDepth>
         <maxVel>0.1</maxVel>
@@ -21,25 +21,25 @@
         <mu1>0.1</mu1>
         <mu2>0.1</mu2>
-        <kp>1e+6</kp>
-        <kd>100</kd>
+        <kp>1000000.0</kp>
+        <kd>100.0</kd>
         <minDepth>0.001</minDepth>
-        <maxVel>0.1</maxVel>
+        <maxVel>1.0</maxVel>
     </gazebo>
     <gazebo reference="caster_read_link">
         <mu1>0.1</mu1>
         <mu2>0.1</mu2>
-        <kp>1e+6</kp>
-        <kd>100</kd>
+        <kp>1000000.0</kp>
+        <kd>100.0</kd>
         <minDepth>0.001</minDepth>
-        <maxVel>0.1</maxVel>
+        <maxVel>1.0</maxVel>
     </gazebo>
     <gazebo>
         <plugin filename="gz_ros2_control-system"
-                name="gz_ros2_control::GazeboSimROS2ControlPlugin">
-                <parameters>$(find spiderbot_controllers)/config/spiderbot_controllers.yaml</parameters>
-            </plugin>
-            <plugin filename="gz-sim-sensors-system" name="gz::sim::systems::Sensors">
-                <render_engine>ogre2</render_engine>
-            </plugin>
+            name="gz_ros2_control::GazeboSimROS2ControlPlugin">
+            <parameters>$(find bumperbot_controllers)/config/bumperbot_controllers.yaml</parameters>
+        </plugin>
+        <plugin filename="gz-sim-sensors-system" name="gz::sim::systems::Sensors">
+            <render_engine>ogre2</render_engine>
+        </plugin>
     </gazebo>
 </robot>

File: src/bumperbot_description/urdf/bumperbot_ros2_control.xacro (robot description, xacro)
@@ -3,5 +3,5 @@
         <xacro:if value="$(arg is_sim)">
             <hardware>
-                <plugin>gz_ros2_control::GazeboSimSystem</plugin>
+                <plugin>gz_ros2_control/GazeboSimSystem</plugin>
             </hardware>
         </xacro:if>

Commit message: aligned with course git repo

File: src/bumperbot_description/urdf/bumperbot.urdf.xacro (robot description, xacro)
@@ -31,4 +31,9 @@
         </collision>
     </link>
+    <joint name="base_joint" type="fixed">
+        <parent link="base_footprint" />
+        <child link="base_link" />
+        <origin xyz="0 0 0.033" rpy="0 0 0" />
+    </joint>
     <link name="wheel_right_link">
         <inertial>
@@ -41,5 +46,5 @@
         </inertial>
         <visual>
-            <origin rpy="-${PI/2} 0 0" xyz="0 0 0" />
+            <origin rpy="${PI/2} 0 0" xyz="0 0 0" />
             <geometry>
                 <mesh filename="package://bumperbot_description/meshes/wheel_right_link.STL" />
@@ -54,5 +59,12 @@
         </collision>
     </link>
-    <link name="wheel_left_link">
+    <joint name="wheel_right_joint" type="continuous">
+        <origin xyz="0 -0.0701101849418637 0" rpy="0 0 0" />
+        <parent link="base_link" />
+        <child link="wheel_right_link" />
+        <axis xyz="0 1 0" />
+    </joint>
+    <link
+        name="wheel_left_link">
         <inertial>
             <origin xyz="0 0.014 0" rpy="0 0 0" />
@@ -64,5 +76,5 @@
         </inertial>
         <visual>
-            <origin rpy="${PI/2} 0 0" xyz="0 0 0" />
+            <origin rpy="-${PI/2} 0 0" xyz="0 0 0" />
             <geometry>
                 <mesh filename="package://bumperbot_description/meshes/wheel_left_link.STL" />
@@ -77,4 +89,10 @@
         </collision>
     </link>
+    <joint name="wheel_left_joint" type="continuous">
+        <origin xyz="0 0.0701101849418642 0" rpy="0 0 0" />
+        <parent link="base_link" />
+        <child link="wheel_left_link" />
+        <axis xyz="0 1 0" />
+    </joint>
     <link name="caster_front_link">
         <inertial>
@@ -100,4 +118,10 @@
         </collision>
     </link>
+    <joint name="caster_front_joint" type="fixed">
+        <origin xyz="0.04755 0 -0.0275" rpy="0 0 0" />
+        <parent link="base_link" />
+        <child link="caster_front_link" />
+        <axis xyz="0 0 0" />
+    </joint>
     <link name="caster_rear_link">
         <inertial>
@@ -123,31 +147,9 @@
         </collision>
     </link>
-    <!-- JOINTS -->
-    <joint name="base_joint" type="fixed">
-        <parent link="base_footprint" />
-        <child link="base_link" />
-        <origin rpy="0 0 0" xyz="0 0 0.033" />
-    </joint>
-    <joint name="wheel_right_joint" type="continuous">
-        <parent link="base_link" />
-        <child link="wheel_right_link" />
-        <origin rpy="0 0 0" xyz="0 0.07 0.0" />
-        <axis xyz="0 1 0" />
-    </joint>
-    <joint name="wheel_left_joint" type="continuous">
-        <parent link="base_link" />
-        <child link="wheel_left_link" />
-        <origin rpy="0 0 0" xyz="0 -0.07 0.0" />
-        <axis xyz="0 1 0" />
-    </joint>
-    <joint name="caster_front_joint" type="fixed">
-        <parent link="base_link" />
-        <child link="caster_front_link" />
-        <origin rpy="0 0 0" xyz="0.04755 0 -0.0275" />
-    </joint>
     <joint name="caster_rear_joint" type="fixed">
+        <origin xyz="-0.04755 0 -0.0275" rpy="0 0 0" />
         <parent link="base_link" />
         <child link="caster_rear_link" />
-        <origin rpy="0 0 0" xyz="-0.04755 0  -0.0275" />
+        <axis xyz="0 0 0" />
     </joint>
 </robot>

Commit message: added lidar to urdf

File: src/bumperbot_description/urdf/bumperbot.urdf.xacro (robot description, xacro)
@@ -9,4 +9,5 @@
     <!-- <xacro:include filename="$(find bumperbot_description)/urdf/can.xacro" /> -->
     <xacro:include filename="$(find bumperbot_description)/urdf/imu.xacro" />
+    <xacro:include filename="$(find bumperbot_description)/urdf/lidar.xacro" />
     <link name="base_footprint" />
     <link name="base_link">

File: src/bumperbot_description/urdf/bumperbot_gazebo.xacro (robot description, xacro)
@@ -93,3 +93,32 @@
         </sensor>
     </gazebo>
+    <gazebo reference="laser_link">
+        <sensor name="lidar" type="gpu_ray">
+            <always_on>true</always_on>
+            <visualize>true</visualize>
+            <topic>scan</topic>
+            <update_rate>5</update_rate>
+            <gz_frame_id>laser_link</gz_frame_id>
+            <ray>
+                <scan>
+                    <horizontal>
+                        <samples>360</samples>
+                        <resolution>1</resolution>
+                        <min_angle>0.0</min_angle>
+                        <max_angle>6.283185307179586</max_angle>
+                    </horizontal>
+                </scan>
+                <range>
+                    <min>0.12</min>
+                    <max>12.0</max>
+                    <resolution>0.02</resolution>
+                </range>
+                <noise>
+                    <type>gaussian</type>
+                    <mean>0.0</mean>
+                    <stddev>0.01</stddev>
+                </noise>
+            </ray>
+        </sensor>
+    </gazebo>
 </robot>

File: src/bumperbot_description/urdf/imu.xacro (robot description, xacro)
@@ -5,8 +5,7 @@
             <origin xyz="-0.00552433659106688 0.000168210391520346 0.000514000497342681" rpy="0 0 0" />
             <mass value="0.000528415362211671" />
-            <inertia ixx="1.46176048428261E-08" ixy="1.40015117949421E-10"
-                ixz="-1.99633872937403E-12"
-                iyy="8.59662482954888E-09" iyz="7.52375112767959E-12"
-                izz="2.30279421279312E-08" />
+            <inertia ixx="1.46176048428261E-08" ixy="1.40015117949421E-10" ixz="-1.99633872937403E-12"
+                     iyy="8.59662482954888E-09" iyz="7.52375112767959E-12"
+                     izz="2.30279421279312E-08" />
         </inertial>
         <visual>
